File: sensor_board.sch (EAGLE design)
At the start: 9 parts, among them J1 2p-2.54, Q1 S8050

Commit message: PCB cosmetic changes
now, READY for sensing to SEEED for v1 fabrication.
Parts:
- added TRIG_ECHO: (no value), SparkFun-Retired:JUMPER-2SMD-NC
Connections:
- net ECHO: now also TRIG_ECHO.2
- net TRIG: now also TRIG_ECHO.1
Changed lines of the file:
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@@
 <?xml version="1.0" encoding="utf-8"?>
 <!DOCTYPE eagle SYSTEM "eagle.dtd">
-<eagle version="7.6.0">
+<eagle version="7.2.0">
 <drawing>
 <settings>
@@
 <layers>
 <layer number="1" name="Top" color="4" fill="1" visible="no" active="no"/>
+<layer number="2" name="Route2" color="1" fill="3" visible="no" active="no"/>
+<layer number="3" name="Route3" color="4" fill="3" visible="no" active="no"/>
+<layer number="4" name="Route4" color="1" fill="4" visible="no" active="no"/>
+<layer number="5" name="Route5" color="4" fill="4" visible="no" active="no"/>
+<layer number="6" name="Route6" color="1" fill="8" visible="no" active="no"/>
+<layer number="7" name="Route7" color="4" fill="8" visible="no" active="no"/>
+<layer number="8" name="Route8" color="1" fill="2" visible="no" active="no"/>
+<layer number="9" name="Route9" color="4" fill="2" visible="no" active="no"/>
+<layer number="10" name="Route10" color="1" fill="7" visible="no" active="no"/>
+<layer number="11" name="Route11" color="4" fill="7" visible="no" active="no"/>
+<layer number="12" name="Route12" color="1" fill="5" visible="no" active="no"/>
+<layer number="13" name="Route13" color="4" fill="5" visible="no" active="no"/>
+<layer number="14" name="Route14" color="1" fill="6" visible="no" active="no"/>
+<layer number="15" name="Route15" color="4" fill="6" visible="no" active="no"/>
 <layer number="16" name="Bottom" color="1" fill="1" visible="no" active="no"/>
 <layer number="17" name="Pads" color="2" fill="1" visible="no" active="no"/>
@@
 <part name="C1" library="adafruit" deviceset="C-US" device="C1206"/>
 <part name="J1" library="Seeed-Connector -2016" deviceset="DIP-BLACK-MALE-HEADER-VERT(2P-2.54)" device="" value="2p-2.54"/>
+<part name="TRIG_ECHO" library="SparkFun-Retired" deviceset="JUMPER-2" device="SMD-NC"/>
 </parts>
 <sheets>
@@
 <instance part="C1" gate="G$1" x="78.74" y="20.32"/>
 <instance part="J1" gate="G$1" x="147.32" y="-2.54"/>
+<instance part="TRIG_ECHO" gate="A" x="147.32" y="-12.7" rot="R270"/>
 </instances>
 <busses>
@@
 <segment>
 <pinref part="J1" gate="G$1" pin="1"/>
-<wire x1="139.7" y1="0" x2="129.54" y2="0" width="0.1524" layer="91"/>
+<wire x1="139.7" y1="0" x2="137.16" y2="0" width="0.1524" layer="91"/>
 <label x="129.54" y="0" size="1.778" layer="95" rot="R180" xref="yes"/>
+<pinref part="TRIG_ECHO" gate="A" pin="1"/>
+<wire x1="137.16" y1="0" x2="129.54" y2="0" width="0.1524" layer="91"/>
+<wire x1="144.78" y1="-12.7" x2="137.16" y2="-12.7" width="0.1524" layer="91"/>
+<wire x1="137.16" y1="-12.7" x2="137.16" y2="0" width="0.1524" layer="91"/>
+<junction x="137.16" y="0"/>
 </segment>
 </net>
@@
 <segment>
 <pinref part="J1" gate="G$1" pin="2"/>
-<wire x1="139.7" y1="-5.08" x2="129.54" y2="-5.08" width="0.1524" layer="91"/>
+<wire x1="139.7" y1="-5.08" x2="134.62" y2="-5.08" width="0.1524" layer="91"/>
 <label x="129.54" y="-5.08" size="1.778" layer="95" rot="R180" xref="yes"/>
+<pinref part="TRIG_ECHO" gate="A" pin="2"/>
+<wire x1="134.62" y1="-5.08" x2="129.54" y2="-5.08" width="0.1524" layer="91"/>
+<wire x1="144.78" y1="-15.24" x2="134.62" y2="-15.24" width="0.1524" layer="91"/>
+<wire x1="134.62" y1="-15.24" x2="134.62" y2="-5.08" width="0.1524" layer="91"/>
+<junction x="134.62" y="-5.08"/>
 </segment>
 </net>
